File: simpleRTK2BpiHAT.kicad_pcb (KiCad board)
At the start: 2 copper layers, 86.4 x 53.3 mm, 17 parts, among them J1 Conn_01x04, J10 Conn_01x04, J11 Conn_01x06, J2 Conn_01x05, J3 Conn_01x07, J4 Conn_01x04, J5 Screw_Terminal_01x02, J6 Raspberry_Pi_2_3, J7 Conn_01x02, J8 Conn_01x04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

Commit message: shutdownSW GND
shutdownSW のGNDがつながってなかった
Routing:
- net GND: track 11.2 -> 15.8 mm
- net GPIO3: track 49.1 -> 50.1 mm
Changed lines of the file:
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@@
     (thickness 1.6)
     (drawings 37)
-    (tracks 163)
+    (tracks 167)
     (zones 0)
     (modules 17)
@@
   (segment (start 155.790002 122.212998) (end 154.178 123.825) (width 0.25) (layer B.Cu) (net 2))
   (segment (start 155.790002 122.047) (end 155.790002 122.212998) (width 0.25) (layer B.Cu) (net 2))
+  (segment (start 161.036 116.078) (end 161.798 116.84) (width 0.25) (layer F.Cu) (net 2))
+  (segment (start 157.48 116.078) (end 161.036 116.078) (width 0.25) (layer F.Cu) (net 2))
   (segment (start 146.53006 123.79706) (end 146.558 123.825) (width 0.25) (layer F.Cu) (net 3))
   (segment (start 141.45006 123.79706) (end 141.478 123.825) (width 0.25) (layer F.Cu) (net 3))
@@
   (segment (start 164.973 114.3) (end 161.798 114.3) (width 0.25) (layer B.Cu) (net 31))
   (segment (start 174.498 123.825) (end 164.973 114.3) (width 0.25) (layer B.Cu) (net 31))
+  (segment (start 157.607 110.871) (end 157.48 110.998) (width 0.25) (layer B.Cu) (net 31))
+  (segment (start 158.369 110.871) (end 157.607 110.871) (width 0.25) (layer B.Cu) (net 31))
   (segment (start 171.958 123.6726) (end 171.958 123.825) (width 0.25) (layer F.Cu) (net 32))
   (segment (start 171.958 123.6726) (end 171.958 123.825) (width 0.25) (layer B.Cu) (net 32))
